File: volt-glitcher/kicad/device.kicad_pcb (KiCad board)
At the start: 4 copper layers, 0 parts

Commit message: feat: rewrite volt-glitcher — full production-quality design
Parts:
- added ?: , Package_QFP:LQFP-100_14x14mm_P0.5mm, F.Cu at (75.0, 55.0)
- added ?: , Package_TO_SOT_SMD:SOT-23-6, F.Cu at (60.0, 115.0)
- added ?: , Package_SO:VSSOP-8_2.3x2mm_P0.5mm, F.Cu at (30.0, 85.0)
- added ?: , Package_SO:VSSOP-8_2.3x2mm_P0.5mm, F.Cu at (30.0, 95.0)
- added ?: , Package_DFN_QFN:DDPAK-7, F.Cu at (30.0, 105.0)
- added ?: , Package_DFN_QFN:DDPAK-7, F.Cu at (30.0, 115.0)
- added ?: , Connector_USB:USB_Micro-B_Molex-105017-0001, F.Cu at (10.0, 55.0)
- added ?: , Connector_PinHeader_2.54mm:PinHeader_2x05_P2.54mm_Vertical, F.Cu at (10.0, 75.0)
- added ?: , Connector_PinHeader_2.54mm:PinHeader_1x06_P2.54mm_Vertical, F.Cu at (165.0, 55.0)
- added ?: , Connector_PinHeader_2.54mm:PinHeader_1x04_P2.54mm_Vertical, F.Cu at (165.0, 75.0)
- added ?: , Connector_PinHeader_2.54mm:PinHeader_1x04_P2.54mm_Vertical, F.Cu at (165.0, 95.0)
- added ?: , Package_QFP:TQFP-144_20x20mm_P0.5mm, F.Cu at (130.0, 55.0)
- added ?: , Connector_Card:microSD_HC_Hirose_DM3BT-DSF-PEJS, F.Cu at (100.0, 10.0)
- added ?: , Crystal:Crystal_SMD_5032-2Pin_5.0x3.2mm, F.Cu at (65.0, 35.0)
- added ?: , Crystal:Crystal_SMD_3215-2Pin_3.2x1.5mm, F.Cu at (65.0, 25.0)
- added ?: , LED_SMD:LED_0805_2012Metric, F.Cu at (90.0, 10.0)
- added ?: , LED_SMD:LED_0805_2012Metric, F.Cu at (100.0, 10.0)
- added ?: , LED_SMD:LED_0805_2012Metric, F.Cu at (110.0, 10.0)
- added ?: , LED_SMD:LED_0805_2012Metric, F.Cu at (120.0, 10.0)
- added ?: , Button_Switch_SMD:SW_Push_1P1T_NO_6x6mm_H9.5mm, F.Cu at (140.0, 10.0)
- added ?: , Button_Switch_SMD:SW_Push_1P1T_NO_4.5x4.5mm, F.Cu at (150.0, 10.0)
- added ?: , Package_SO:VSSOP-8_2.3x2mm_P0.5mm, F.Cu at (45.0, 85.0)
- added ?: , Package_TO_SOT_SMD:SuperSOT-6, F.Cu at (45.0, 95.0)
- added ?: , Package_TO_SOT_SMD:SOT-23, F.Cu at (45.0, 105.0)
- added ?: , Package_TO_SOT_SMD:SOT-23, F.Cu at (45.0, 115.0)
- added ?: , Package_DFN_QFN:DFN-8-1EP_2x2mm_P0.5mm, F.Cu at (60.0, 85.0)
- added ?: , Package_SO:TSSOP-8_4.4x3mm_P0.65mm, F.Cu at (60.0, 95.0)
- added ?: , Package_SO:SOIC-8_3.9x4.9mm_P1.27mm, F.Cu at (60.0, 105.0)
Routing:
- net GLITCH_CLK: track 0.00 -> 128.2 mm
- net GLITCH_SHUNT: track 0.00 -> 126.5 mm
- net GLITCH_EM: track 0.00 -> 126.5 mm
- net SPI1_SCK: track 0.00 -> 55.0 mm
- net SPI1_NSS: track 0.00 -> 55.0 mm
- net SPI1_MOSI: track 0.00 -> 55.0 mm
- net SPI1_MISO: track 0.00 -> 55.0 mm
Other:
- net class Glitch added: clearance 0.3, trace_width 1.0, via_dia 1.0, via_drill 0.6
- net class Power added: clearance 0.2, trace_width 0.4, via_dia 0.8, via_drill 0.4
- net class RF added: clearance 0.15, trace_width 0.2, via_dia 0.5, via_drill 0.25
- net class Signal added: clearance 0.15, trace_width 0.15, via_dia 0.6, via_drill 0.3
- board text added: "Hacker Devices 2026"
- board text added: "VoltGlitcher Pro v1.0"
