File: volt-glitcher/kicad/device.kicad_sch (KiCad schematic)
At the start: 0 parts

Commit message: feat: rewrite volt-glitcher — full production-quality design
Parts:
- added ?: (no value), symbol Connector:MicroSD
Other:
- company: (none) -> Hacker Devices
- title: (none) -> VoltGlitcher Pro - Voltage Glitch Injection Tool
